File: Tic-tac-toe_Business_Card.kicad_pcb (KiCad board)
At the start: 2 copper layers, 85 x 55 mm, 79 parts, among them J1 USB_C_Receptacle_USB2.0_14P, J2 Conn_01x04, SW1 SW_Push, SW2 SW_Push, SW3 SW_Push, U1 MCP1700x-330xxTT, U2 NT3H2111W0FHKH, U3 RP2040, U4 W25Q16JVUXIQ TR, Y1 12 MHz

Commit message: Update Readme
Parts:
- removed the C8 at (161.7, 93.8)
- removed the D1 at (158.6, 103.5)
- removed the R21 at (128.0, 79.1)
- removed the R9 at (158.6, 101.6)
- removed U2: NT3H2111W0FHKH, NFC_Tic_Tac_Toe:XQFN-8_L1.6-W1.6-P0.50-BL_NT3H2111W0FHKH
- added C4: 1uF, Capacitor_SMD:C_0402_1005Metric, F.Cu at (91.5, 61.9)
- added G***: LOGO, image:nfc, F.Cu at (38.8, 35.9)
- added G***: LOGO, image:nfc, F.Cu at (38.8, 60.3)
- added G***: LOGO, image:stem_logo, F.Cu at (38.6, 48.0)
- added G***: LOGO, image:back_image, B.Cu at (64.9, 46.2)
- added R24: 1K, Resistor_SMD:R_0402_1005Metric, F.Cu at (57.0, 46.5)
- added U5: NT3H2111W0FHKH, NFC_Tic_Tac_Toe:XQFN-8_L1.6-W1.6-P0.50-BL_NT3H2111W0FHKH, F.Cu at (54.7, 47.4)
- D13: footprint LED_SMD:LED_0603_1608Metric -> LED_SMD:LED_0402_1005Metric
- R25: renamed from R10; value 100 -> 330
- R26: renamed from R11; value 470 -> 1k
- moved C11 77.1 mm to (79.8, 59.0)
- moved C12 77.1 mm to (80.9, 67.0)
- moved C15 77.1 mm to (90.9, 59.5)
- moved C17 77.1 mm to (79.2, 68.0)
- moved C6 77.1 mm to (91.5, 56.8)
- moved C7 77.1 mm to (91.2, 60.6)
- moved L1 77.1 mm to (38.3, 48.0)
- moved R1 77.1 mm to (89.7, 54.8)
- moved R6 77.1 mm to (93.1, 57.9)
- moved R7 77.1 mm to (93.6, 58.9)
- moved SW3 77.1 mm to (64.4, 65.1)
- moved U4 77.1 mm to (85.1, 61.7)
- moved C1 77.1 mm to (91.5, 54.4)
- moved C13 77.1 mm to (79.8, 64.2)
- moved C14 77.1 mm to (90.2, 56.6)
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- renumbered C3 to C1, C14 to C11, C15 to C12, C16 to C13, C4 to C14, C5 to C15, C6 to C16, C1 to C2, C2 to C3, C9 to C6, C10 to C7, C11 to C8, C12 to C9, D4 to D1, D22 to D10, D23 to D11, D24 to D12, D25 to D14, D26 to D15, D27 to D16, D2 to D17, D3 to D18, D28 to D19, D5 to D2, D29 to D20, D30 to D21, D6 to D3, D7 to D4, D8 to D5, D9 to D6, D10 to D7, D11 to D8, D12 to D9, R3 to R1, R14 to R10, R8 to R11, R15 to R12, R16 to R13, R17 to R14, R18 to R15, R19 to R16, R20 to R17, R30 to R18, R31 to R19, R4 to R2, R32 to R20, R33 to R21, R34 to R22, R35 to R23, R36 to R27, R37 to R28, R38 to R29, R1 to R3, R2 to R4, R12 to R8, R13 to R9, U4 to U3, U3 to U4
Connections:
- net GPIO14 renamed Net-(U4-GPIO14)
- net GPIO15 renamed Net-(U4-GPIO15)
- U4 pad 28: GPIO17 -> unconnected-(U4-GPIO17-Pad28)
Routing:
- net Net-(U5-LA): track 0.00 -> 7.06 mm, vias 0 -> 1
- net GPIO17: track 5.14 -> 0.00 mm
- net Net-(D1-A) (its old number): track 2.05 -> 0.00 mm
- net Net-(U5-LB): track 0.00 -> 1.83 mm
- net +3V3: track 72.7 -> 71.0 mm
- net Net-(U2-LB): track 1.37 -> 0.00 mm
- net SWCLK: track 12.2 -> 11.1 mm
- net SWD: track 12.3 -> 11.2 mm
- net Net-(D13-K): track 4.27 -> 5.14 mm
- net Net-(U5-VCC): track 4.89 -> 5.75 mm
- net Net-(D13-A): track 2.25 -> 1.67 mm
- net GND: track 35.1 -> 35.6 mm, vias 31 -> 29
Other:
- board text added: "By Hung-Chi"
- board text added: "Next"
- board text added: "Select"
- board text added: "Tic-Tac-Toe"

Commit message: Update Repo
Parts:
- C13, C17: value 33pF -> 15pF
- moved C2 0.53 mm to (95.8, 67.3)
- moved C3 0.14 mm to (92.7, 64.3)
Changed lines of the file:
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@@
 	(footprint "Capacitor_SMD:C_0603_1608Metric"
 		(layer "F.Cu")
-		(at 95.843359 66.77 180)
+		(at 95.843359 67.3 180)
 		(descr "Capacitor SMD 0603 (1608 Metric), square (rectangular) end terminal, IPC-7351 nominal, (Body size source: IPC-SM-782 page 76, https://www.pcb-3d.com/wordpress/wp-content/uploads/ipc-sm-782a_amendment_1_and_2.pdf), generated with kicad-footprint-generator")
 		(tags "capacitor")
@@
 	(footprint "Capacitor_SMD:C_0603_1608Metric"
 		(layer "F.Cu")
-		(at 92.843359 64.27 90)
+		(at 92.7 64.27 90)
 		(descr "Capacitor SMD 0603 (1608 Metric), square (rectangular) end terminal, IPC-7351 nominal, (Body size source: IPC-SM-782 page 76, https://www.pcb-3d.com/wordpress/wp-content/uploads/ipc-sm-782a_amendment_1_and_2.pdf), generated with kicad-footprint-generator")
 		(tags "capacitor")
@@
 			)
 		)
-		(property "Value" "33pF"
+		(property "Value" "15pF"
 			(at 0 1.16 45)
 			(layer "F.Fab")
@@
 			)
 		)
-		(property "Value" "33pF"
+		(property "Value" "15pF"
 			(at 0 1.16 135)
 			(layer "F.Fab")
@@
 	)
 	(segment
+		(start 92.6 65.045)
+		(end 92.6 65.3)
+		(width 0.2)
+		(layer "F.Cu")
+		(net 3)
+	)
+	(segment
 		(start 80.960275 59.02)
 		(end 81.936702 59.996427)
@@
 	)
 	(segment
+		(start 92.775 65.22)
+		(end 92.6 65.045)
+		(width 0.2)
+		(layer "F.Cu")
+		(net 3)
+	)
+	(segment
 		(start 89.870489 55.140624)
 		(end 89.083816 55.927297)
@@
 	)
 	(segment
-		(start 94.905859 65.22)
-		(end 93.018359 65.22)
-		(width 0.3)
-		(layer "F.Cu")
-		(net 3)
-	)
-	(segment
 		(start 91.045859 61.95)
 		(end 89.344403 61.95)
@@
 	)
 	(segment
-		(start 92.843359 69.3975)
-		(end 93.165859 69.72)
-		(width 0.3)
-		(layer "F.Cu")
-		(net 3)
-	)
-	(segment
 		(start 84.912878 57.365252)
 		(end 84.567877 57.365252)
@@
 	)
 	(segment
+		(start 92.6 65.3)
+		(end 93.165859 65.865859)
+		(width 0.2)
+		(layer "F.Cu")
+		(net 3)
+	)
+	(segment
 		(start 82.151403 64.925928)
 		(end 82.151403 65.258542)
@@
 	)
 	(segment
-		(start 93.018359 65.22)
-		(end 92.843359 65.045)
-		(width 0.3)
-		(layer "F.Cu")
-		(net 3)
-	)
-	(segment
 		(start 82.78523 64.292101)
 		(end 82.151403 64.925928)
@@
 	)
 	(segment
+		(start 93.165859 65.865859)
+		(end 93.165859 69.72)
+		(width 0.2)
+		(layer "F.Cu")
+		(net 3)
+	)
+	(segment
 		(start 84.850782 57.819339)
 		(end 84.850782 58.112603)
@@
 	)
 	(segment
+		(start 93.1 69.654141)
+		(end 93.165859 69.72)
+		(width 0.2)
+		(layer "F.Cu")
+		(net 3)
+	)
+	(segment
 		(start 90.556082 57.119411)
 		(end 90.556082 57.2044)
@@
 	)
 	(segment
-		(start 92.843359 65.045)
-		(end 92.843359 69.3975)
-		(width 0.3)
-		(layer "F.Cu")
-		(net 3)
-	)
-	(segment
 		(start 90.556082 57.119411)
 		(end 91.116448 57.119411)
@@
 		(layer "F.Cu")
 		(net 3)
+	)
+	(segment
+		(start 94.905859 65.22)
+		(end 92.775 65.22)
+		(width 0.2)
+		(layer "F.Cu")
+		(net 3)
